Commit message: Refactor code structure for improved readability and maintainability

File: src/test/testdata/simple_test.urdf (robot description, URDF)
Before this commit: robot simple_test_robot, 2 links, 1 joints
Links:
- added link front_left_wheel; visual cylinder length=0.05 radius=0.15
- added link front_right_wheel; visual cylinder length=0.05 radius=0.15
- added link rear_left_wheel; visual cylinder length=0.05 radius=0.15
- added link rear_right_wheel; visual cylinder length=0.05 radius=0.15
Joints:
- added joint front_left_wheel_joint: type continuous, parent base_link, child front_left_wheel, origin xyz=0.575 0.575 -0.65 rpy=1.57 0 0, axis 0 0 1
- added joint front_right_wheel_joint: type continuous, parent base_link, child front_right_wheel, origin xyz=0.575 -0.575 -0.65 rpy=1.57 0 0, axis 0 0 1
- added joint rear_left_wheel_joint: type continuous, parent base_link, child rear_left_wheel, origin xyz=-0.575 0.575 -0.65 rpy=1.57 0 0, axis 0 0 1
- added joint rear_right_wheel_joint: type continuous, parent base_link, child rear_right_wheel, origin xyz=-0.575 -0.575 -0.65 rpy=1.57 0 0, axis 0 0 1
