Commit message: Update src/test/testdata/axis_test.urdf
Co-authored-by: Copilot <175728472+Copilot@users.noreply.github.com>

File: src/test/testdata/axis_test.urdf (robot description, URDF)
Before this commit: robot axis_test, 4 links, 3 joints
Joints:
- joint y_axis_joint: origin xyz=0.0 .5 0.0 rpy=0 0 0 -> xyz=0.0 0.5 0.0 rpy=0 0 0
